File: KiCad_and_production_files/JX2_connections.kicad_sch (KiCad schematic)
At the start: 23 parts, among them J4 Conn_02x19_Top_Bottom, Q2 BSS138, SW1 SW_MEC_5E

Commit message: Components rotation offsets added
Parts:
- Q2: JLCPCB Rotation Offset (none) -> -180
Changed lines of the file:
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@@
+      (effects (font (size 1.27 1.27)) hide)
+    )
+    (property "JLCPCB Rotation Offset" "-180" (at 50.8 30.48 0)
       (effects (font (size 1.27 1.27)) hide)
     )
@@
       (effects (font (size 1.27 1.27)) hide)
     )
+    (property "JLCPCB Rotation Offset" "-180" (at 96.52 30.48 0)
+      (effects (font (size 1.27 1.27)) hide)
+    )
