File: KiCad_and_production_files/MicroZed_carrier_board_v4.kicad_sch (KiCad schematic)
At the start: 52 parts, among them CON1 USB_B_Micro, J1 Screw_Terminal_01x02, Q2 BSS138, SW3 SW_SPDT, U1 AP331A, U2 TL431A PJSEMI

Commit message: Components rotation offsets added
Parts:
- D5, D8, Q2, U2: JLCPCB Rotation Offset (none) -> -180
Changed lines of the file:
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@@
+      (effects (font (size 1.27 1.27)) hide)
+    )
+    (property "JLCPCB Rotation Offset" "-180" (at 53.34 128.27 0)
       (effects (font (size 1.27 1.27)) hide)
     )
@@
       (effects (font (size 1.27 1.27)) hide)
     )
+    (property "JLCPCB Rotation Offset" "-180" (at 121.92 81.28 90)
+      (effects (font (size 1.27 1.27)) hide)
+    )
     (pin "1")
     (pin "2")
@@
     )
     (property "LCSC" "C37704" (at 58.42 156.21 0)
+      (effects (font (size 1.27 1.27)) hide)
+    )
+    (property "JLCPCB Rotation Offset" "-180" (at 58.42 156.21 90)
       (effects (font (size 1.27 1.27)) hide)
     )
@@
       (effects (font (size 1.27 1.27)) hide)
     )
+    (property "JLCPCB Rotation Offset" "-180" (at 154.94 104.14 90)
+      (effects (font (size 1.27 1.27)) hide)
+    )
