File: KiCad_and_production_files/UART2USB.kicad_sch (KiCad schematic)
At the start: 11 parts, among them CON1 UART, U5 CH340G, U6 74LVC1G08, Y1 12MHz

Commit message: Components rotation offsets added
Parts:
- U5: JLCPCB Rotation Offset (none) -> 270
Changed lines of the file:
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@@
+      (effects (font (size 1.27 1.27)) hide)
+    )
+    (property "JLCPCB Rotation Offset" "270" (at 91.44 66.04 0)
       (effects (font (size 1.27 1.27)) hide)
     )
